File: PCBs/LowerBoard_r1.sch (EAGLE design)
At the start: 14 parts, among them K1 G2R2, P1 HEADER_5X2, Q1 2N7000

Commit message: finished eagle file for lower PCB
Parts:
- removed COMMUNICATION: 8x1F-H8.5, SmartPrj:PINHD-1X8
- added COMMS: (no value), LowerBoard_r1:PINHD-1X8
- ANALOG, POWER, PWML: device SmartPrj:PINHD-1X8 -> LowerBoard_r1:PINHD-1X8
- LEFT_MOTR, RIGHT_MOTR: device con-lsta:FE06-1 -> LowerBoard_r1:FE06-1
- P1: device myDevices:HEADER_5X2 -> LowerBoard_r1:HEADER_5X2
- PWMH: device SmartPrj:PINHD-1X10 -> LowerBoard_r1:PINHD-1X10
- U$11, U$12: device myDevices:TB2 -> LowerBoard_r1:TB2
- U$5: device myDevices:POLOLU_MINIIMU9_V2 -> LowerBoard_r1:POLOLU_MINIIMU9_V2
Connections:
- net SCL0: now also COMMS.8; no longer COMMUNICATION.8
- net SDA0: now also COMMS.7; no longer COMMUNICATION.7
- net XBEE_DIN: now also COMMS.1; no longer COMMUNICATION.1
- net XBEE_DOUT: now also COMMS.2; no longer COMMUNICATION.2
